File: M921-SS.kicad_pcb (KiCad board)
At the start: 2 copper layers, 45.7 x 25.4 mm, 12 parts, among them J1 PIEZZO, J2 A/D CONV

Commit message: Rev.1 PCBGOGO ordering data
Other:
- board text added: "HOLLY&CO.,LTD. 2021 M921-SS Rev.1"
- board text removed: "HOLLY&CO.,LTD. 2021 M921-SS"

Commit message: KiCAD v8
Other:
- net class Default removed
