File: M921-SS.kicad_sch (KiCad schematic)
At the start: 8 parts

Commit message: sche: KiCAD new version
Parts:
- C1, C2, C3: value (none) -> 10uF/50V; footprint (none) -> Capacitor_THT:CP_Radial_D5.0mm_P2.00mm
- D1, D2, D3: value (none) -> MB10M; footprint (none) -> HOLLY_LIB:MB10M
- J1: value (none) -> PIEZZO; footprint (none) -> Connector_JST:JST_XH_B6B-XH-A_1x06_P2.50mm_Vertical
- J2: value (none) -> A/D CONV; footprint (none) -> Connector_JST:JST_XH_B4B-XH-A_1x04_P2.50mm_Vertical
Changed lines of the file:
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@@
     (in_bom yes) (on_board yes)
     (property "Reference" "J1" (id 0) (at 57.3532 70.3326 0))
-    (property "Value" "" (id 1) (at 57.3532 72.644 0))
-    (property "Footprint" "" (id 2) (at 54.61 80.01 0)
+    (property "Value" "PIEZZO" (id 1) (at 57.3532 72.644 0))
+    (property "Footprint" "Connector_JST:JST_XH_B6B-XH-A_1x06_P2.50mm_Vertical" (id 2) (at 54.61 80.01 0)
       (effects (font (size 1.27 1.27)) hide)
     )
@@
       (effects (font (size 1.27 1.27)) (justify left))
     )
-    (property "Value" "" (id 1) (at 111.6076 57.023 0)
-      (effects (font (size 1.27 1.27)) (justify left))
-    )
-    (property "Footprint" "" (id 2) (at 106.68 52.705 0)
+    (property "Value" "MB10M" (id 1) (at 111.6076 57.023 0)
+      (effects (font (size 1.27 1.27)) (justify left))
+    )
+    (property "Footprint" "HOLLY_LIB:MB10M" (id 2) (at 106.68 52.705 0)
       (effects (font (size 1.27 1.27)) (justify left) hide)
     )
@@
       (effects (font (size 1.27 1.27)) (justify left))
     )
-    (property "Value" "" (id 1) (at 111.6076 82.423 0)
-      (effects (font (size 1.27 1.27)) (justify left))
-    )
-    (property "Footprint" "" (id 2) (at 106.68 78.105 0)
+    (property "Value" "MB10M" (id 1) (at 111.6076 82.423 0)
+      (effects (font (size 1.27 1.27)) (justify left))
+    )
+    (property "Footprint" "HOLLY_LIB:MB10M" (id 2) (at 106.68 78.105 0)
       (effects (font (size 1.27 1.27)) (justify left) hide)
     )
@@
       (effects (font (size 1.27 1.27)) (justify left))
     )
-    (property "Value" "" (id 1) (at 111.6076 107.823 0)
-      (effects (font (size 1.27 1.27)) (justify left))
-    )
-    (property "Footprint" "" (id 2) (at 106.68 103.505 0)
+    (property "Value" "MB10M" (id 1) (at 111.6076 107.823 0)
+      (effects (font (size 1.27 1.27)) (justify left))
+    )
+    (property "Footprint" "HOLLY_LIB:MB10M" (id 2) (at 106.68 103.505 0)
       (effects (font (size 1.27 1.27)) (justify left) hide)
     )
@@
       (effects (font (size 1.27 1.27)) (justify left))
     )
-    (property "Value" "" (id 1) (at 137.6172 57.023 0)
-      (effects (font (size 1.27 1.27)) (justify left))
-    )
-    (property "Footprint" "" (id 2) (at 135.5852 59.69 0)
+    (property "Value" "10uF/50V" (id 1) (at 137.6172 57.023 0)
+      (effects (font (size 1.27 1.27)) (justify left))
+    )
+    (property "Footprint" "Capacitor_THT:CP_Radial_D5.0mm_P2.00mm" (id 2) (at 135.5852 59.69 0)
       (effects (font (size 1.27 1.27)) hide)
     )
@@
       (effects (font (size 1.27 1.27)) (justify left))
     )
-    (property "Value" "" (id 1) (at 137.6172 82.423 0)
-      (effects (font (size 1.27 1.27)) (justify left))
-    )
-    (property "Footprint" "" (id 2) (at 135.5852 85.09 0)
+    (property "Value" "10uF/50V" (id 1) (at 137.6172 82.423 0)
+      (effects (font (size 1.27 1.27)) (justify left))
+    )
+    (property "Footprint" "Capacitor_THT:CP_Radial_D5.0mm_P2.00mm" (id 2) (at 135.5852 85.09 0)
       (effects (font (size 1.27 1.27)) hide)
     )
@@
       (effects (font (size 1.27 1.27)) (justify left))
     )
-    (property "Value" "" (id 1) (at 137.6172 107.823 0)
-      (effects (font (size 1.27 1.27)) (justify left))
-    )
-    (property "Footprint" "" (id 2) (at 135.5852 110.49 0)
+    (property "Value" "10uF/50V" (id 1) (at 137.6172 107.823 0)
+      (effects (font (size 1.27 1.27)) (justify left))
+    )
+    (property "Footprint" "Capacitor_THT:CP_Radial_D5.0mm_P2.00mm" (id 2) (at 135.5852 110.49 0)
       (effects (font (size 1.27 1.27)) hide)
     )
@@
       (effects (font (size 1.27 1.27)) (justify right))
     )
-    (property "Value" "" (id 1) (at 169.6212 82.9818 0)
+    (property "Value" "A/D CONV" (id 1) (at 169.6212 82.9818 0)
       (effects (font (size 1.27 1.27)) (justify right))
     )
-    (property "Footprint" "" (id 2) (at 168.91 80.01 0)
+    (property "Footprint" "Connector_JST:JST_XH_B4B-XH-A_1x04_P2.50mm_Vertical" (id 2) (at 168.91 80.01 0)
       (effects (font (size 1.27 1.27)) hide)
     )
@@
       (effects (font (size 1.27 1.27)) hide)
     )
-    (property "Value" "" (id 1) (at 134.747 66.6242 0))
+    (property "Value" "GND" (id 1) (at 134.747 66.6242 0))
     (property "Footprint" "" (id 2) (at 134.62 62.23 0)
       (effects (font (size 1.27 1.27)) hide)
@@
       (effects (font (size 1.27 1.27)) hide)
     )
-    (property "Value" "" (id 1) (at 95.377 70.4342 0))
+    (property "Value" "GND" (id 1) (at 95.377 70.4342 0))
     (property "Footprint" "" (id 2) (at 95.25 66.04 0)
       (effects (font (size 1.27 1.27)) hide)
@@
       (effects (font (size 1.27 1.27)) hide)
     )
-    (property "Value" "" (id 1) (at 134.747 93.2942 0))
+    (property "Value" "GND" (id 1) (at 134.747 93.2942 0))
     (property "Footprint" "" (id 2) (at 134.62 88.9 0)
       (effects (font (size 1.27 1.27)) hide)
@@
       (effects (font (size 1.27 1.27)) hide)
     )
-    (property "Value" "" (id 1) (at 95.377 95.8342 0))
+    (property "Value" "GND" (id 1) (at 95.377 95.8342 0))
     (property "Footprint" "" (id 2) (at 95.25 91.44 0)
       (effects (font (size 1.27 1.27)) hide)
@@
       (effects (font (size 1.27 1.27)) hide)
     )
-    (property "Value" "" (id 1) (at 95.377 121.2342 0))
+    (property "Value" "GND" (id 1) (at 95.377 121.2342 0))
     (property "Footprint" "" (id 2) (at 95.25 116.84 0)
       (effects (font (size 1.27 1.27)) hide)
@@
       (effects (font (size 1.27 1.27)) hide)
     )
-    (property "Value" "" (id 1) (at 134.747 118.6942 0))
+    (property "Value" "GND" (id 1) (at 134.747 118.6942 0))
     (property "Footprint" "" (id 2) (at 134.62 114.3 0)
       (effects (font (size 1.27 1.27)) hide)
@@
       (effects (font (size 1.27 1.27)) hide)
     )
-    (property "Value" "" (id 1) (at 161.417 92.0242 0))
+    (property "Value" "GND" (id 1) (at 161.417 92.0242 0))
     (property "Footprint" "" (id 2) (at 161.29 87.63 0)
       (effects (font (size 1.27 1.27)) hide)
